File: mppt charger/mppt charger.kicad_pcb (KiCad board)
At the start: 2 copper layers, 24 parts, among them U1 LM2576T-ADJ, U2 X9C103P, U3 SC0915, U4 MCP601-xP

Commit message: added output terminal
Parts:
- added Jout1: Screw_Terminal_01x02, TerminalBlock:TerminalBlock_bornier-2_P5.08mm, F.Cu at (147.0, 58.0)
Routing:
- net Vout: track 97.9 -> 125.4 mm
- net Net-(D1-Pad1): track 37.2 -> 45.4 mm

Commit message: version sent for manufacture
Parts:
- added 1k3: 1k3, Resistor_THT:R_Axial_DIN0207_L6.3mm_D2.5mm_P10.16mm_Horizontal, F.Cu at (123.0, 60.0)
- added 9k1: 9k1, Resistor_THT:R_Axial_DIN0207_L6.3mm_D2.5mm_P10.16mm_Horizontal, F.Cu at (133.1, 64.8)
- moved 8k2 4.49 mm to (115.2, 69.1)
- moved 1k8 2.80 mm to (119.0, 61.6)
- moved Cout1 2.54 mm to (80.6, 36.2)
- renumbered R1 to 1k8, R2 to 3k9, R3 to 8k2
Connections:
- U3 pad 34: unconnected-(U3-Pad34) -> VinSense
- U3 pad 39: unconnected-(U3-Pad39) -> Vout
Routing:
- net Net-(Cin1-Pad1): track 21.9 -> 106.3 mm
- net VinSense: track 0.00 -> 30.5 mm
- net Net-(Rf1-Pad1): track 88.3 -> 105.6 mm
- net Vout: track 125.4 -> 134.2 mm
- net Net-(R1-Pad1): track 13.8 -> 10.8 mm
- net +BATT: track 94.2 -> 92.4 mm
