File: mppt charger/mppt charger.kicad_sch (KiCad schematic)
At the start: 20 parts, among them U1 LM2576T-ADJ, U2 X9C103P, U3 SC0915, U4 MCP601-xP

Commit message: added output terminal
Parts:
- added Jout1: Screw_Terminal_01x02, TerminalBlock:TerminalBlock_bornier-2_P5.08mm, symbol Connector:Screw_Terminal_01x02
Connections:
- net GND: now also Jout1.1 (Pin_1)
- net Vout: now also Jout1.2 (Pin_2)
Changed lines of the file:
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@@
+    )
+  )
+  (global_label "Vout" (shape input) (at 271.78 81.28 180) (fields_autoplaced)
+    (effects (font (size 1.27 1.27)) (justify right))
+    (property "Intersheet References" "${INTERSHEET_REFS}" (id 0) (at 265.2545 81.2006 0)
+      (effects (font (size 1.27 1.27)) (justify right) hide)
     )
   )
@@
     )
     (pin "1")
+  )
+  (symbol (lib_id "Connector:Screw_Terminal_01x02") (at 276.86 83.82 0) (mirror x) (unit 1)
+    (in_bom yes) (on_board yes) (fields_autoplaced)
+    (property "Reference" "Jout1" (id 0) (at 276.86 74.93 0))
+    (property "Value" "Screw_Terminal_01x02" (id 1) (at 276.86 77.47 0))
+    (property "Footprint" "TerminalBlock:TerminalBlock_bornier-2_P5.08mm" (id 2) (at 276.86 83.82 0)
+      (effects (font (size 1.27 1.27)) hide)
+    )
+    (property "Datasheet" "~" (id 3) (at 276.86 83.82 0)
+      (effects (font (size 1.27 1.27)) hide)
+    )
+    (pin "1")
+    (pin "2")
   )
   (symbol (lib_id "Device:R") (at 220.98 95.25 180) (unit 1)
@@
     (pin "1")
   )
+  (symbol (lib_id "power:GND") (at 271.78 83.82 0) (unit 1)
+    (in_bom yes) (on_board yes) (fields_autoplaced)
+    (property "Reference" "#PWR0117" (id 0) (at 271.78 90.17 0)
+      (effects (font (size 1.27 1.27)) hide)
+    )
+    (property "Value" "GND" (id 1) (at 271.78 88.9 0))
+    (property "Footprint" "" (id 2) (at 271.78 83.82 0)
+      (effects (font (size 1.27 1.27)) hide)
+    )
+    (property "Datasheet" "" (id 3) (at 271.78 83.82 0)
+      (effects (font (size 1.27 1.27)) hide)
+    )
+    (pin "1")
+  )
   (symbol (lib_id "power:-BATT") (at 38.1 107.95 0) (mirror x) (unit 1)
     (in_bom yes) (on_board yes) (fields_autoplaced)
@@
       (reference "#PWR0116") (unit 1) (value "GND") (footprint "")
     )
+    (path "/dc08c6c7-93e9-4580-b87f-3463dca50515"
+      (reference "#PWR0117") (unit 1) (value "GND") (footprint "")
+    )
     (path "/7395de6f-6f04-4949-bbb2-d6ba4f5c1c78"
       (reference "Cin1") (unit 1) (value "100uF") (footprint "Capacitor_THT:CP_Radial_D8.0mm_P5.00mm")
@@
       (reference "Jin1") (unit 1) (value "Screw_Terminal_01x02") (footprint "TerminalBlock:TerminalBlock_bornier-2_P5.08mm")
     )
+    (path "/14e1b2a0-bf13-495d-b056-57752aff2703"
+      (reference "Jout1") (unit 1) (value "Screw_Terminal_01x02") (footprint "TerminalBlock:TerminalBlock_bornier-2_P5.08mm")
+    )
     (path "/db114e00-fbd1-4e76-a26c-829092f18086"

Commit message: version sent for manufacture
Parts:
- added R4: 9k1, Resistor_THT:R_Axial_DIN0207_L6.3mm_D2.5mm_P10.16mm_Horizontal, symbol Device:R
- added R5: 1k3, Resistor_THT:R_Axial_DIN0207_L6.3mm_D2.5mm_P10.16mm_Horizontal, symbol Device:R
Connections:
- net GND: now also R5.1
- net Vout: now also U3.39 (VSYS)
- net at Cin1.1, Jin1.1 (Pin_1), U1.1 (VIN): now also R4.2
- net VinSense: now reaches U3.34 (GP28)
- net VinSense: now also R4.1, R5.2
Other:
- moved on the sheet: Cin1, H1, H2
